Commit message: fix package path error

File: ros_ws/src/maxbot_sim/urdf/lidar.urdf.xacro (robot description, xacro)
@@ -8,5 +8,5 @@
             <origin rpy="0 0 0" xyz="0 0 0"/>
             <geometry>
-                <mesh filename="package://maxbot/meshes/hokuyo.dae"/>
+                <mesh filename="package://maxbot_sim/meshes/hokuyo.dae"/>
             </geometry>
         </visual>
